Commit message: Add TP5 pick-and-place pipeline

File: bcr_ws/src/bcr_arm_description/urdf/robots/bcr_arm.urdf.xacro (robot description, xacro)
@@ -29,5 +29,5 @@
   <xacro:if value="$(arg use_camera)">
     <xacro:include filename="$(find bcr_arm_description)/urdf/sensors/depth_camera.urdf.xacro"/>
-    <xacro:depth_camera prefix="$(arg prefix)" parent_link="flange"/>
+    <xacro:depth_camera prefix="$(arg prefix)" parent_link="world" xyz="0.6 0 1.2" rpy="0 1.5708 0"/>
   </xacro:if>
   <!-- ROS2 Control -->

File: bcr_ws/src/bcr_arm_description/urdf/sensors/depth_camera.urdf.xacro (robot description, xacro)
@@ -1,10 +1,10 @@
 <?xml version="1.0"?>
 <robot xmlns:xacro="http://www.ros.org/wiki/xacro">
-  <xacro:macro name="depth_camera" params="prefix parent_link namespace:=bcr_arm">
-    <!-- Camera Mount and Link -->
+  <xacro:macro name="depth_camera" params="prefix parent_link xyz rpy namespace:=bcr_arm">
+    <!-- Fixed RGB-D camera support. For TP5 this is mounted above the table. -->
     <joint name="${prefix}camera_mount_joint" type="fixed">
       <parent link="${parent_link}"/>
       <child link="${prefix}camera_base_link"/>
-      <origin xyz="0.04 0 0.096125" rpy="0 0 0"/>
+      <origin xyz="${xyz}" rpy="${rpy}"/>
     </joint>
     <link name="${prefix}camera_base_link">
@@ -29,5 +29,4 @@
       <parent link="${prefix}camera_base_link"/>
       <child link="${prefix}camera_link"/>
-      <!-- Pointing forward from the mount -->
       <origin xyz="0.0125 0 0" rpy="0 0 0"/>
     </joint>
@@ -41,12 +40,15 @@
     </joint>
     <link name="${prefix}camera_depth_optical_frame"/>
-    <!-- Ignition Gazebo Camera Plugin -->
+    <!-- Gazebo RGB-D camera. With topic /camera, Gazebo publishes:
+         /camera/image, /camera/depth_image, /camera/points, and /camera/camera_info. -->
     <gazebo reference="${prefix}camera_link">
-      <sensor type="camera" name="depth_camera">
+      <sensor type="rgbd_camera" name="depth_camera">
         <always_on>true</always_on>
         <update_rate>20</update_rate>
         <visualize>true</visualize>
+        <topic>/camera</topic>
         <camera>
-          <horizontal_fov>1.0</horizontal_fov>
+          <camera_info_topic>/camera/camera_info</camera_info_topic>
+          <horizontal_fov>1.047</horizontal_fov>
           <image>
             <width>640</width>
@@ -58,7 +60,14 @@
             <height>480</height>
           </depth_image>
+          <depth_camera>
+            <output>points</output>
+            <clip>
+              <near>0.1</near>
+              <far>5.0</far>
+            </clip>
+          </depth_camera>
           <clip>
             <near>0.1</near>
-            <far>10.0</far>
+            <far>5.0</far>
           </clip>
         </camera>
